File: pcb_data/Assemble_L/Assemble_L.kicad_sch (KiCad schematic)
At the start: 75 parts, among them U1 XIAO-nRF52840

Commit message: update foot print reference, and fix GND filling area DRC error
Parts:
- U1: footprint Module:MOUDLE14P-XIAO-DIP-SMD -> Seeed Studio XIAO Series Library:XIAO-nRF52840-DIP
Changed lines of the file:
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@@
 			)
 		)
-		(property "Footprint" "Module:MOUDLE14P-XIAO-DIP-SMD"
+		(property "Footprint" "Seeed Studio XIAO Series Library:XIAO-nRF52840-DIP"
 			(at 232.41 80.264 0)
 			(effects

Commit message: complete to design pattern of board L
Parts:
- U1: footprint Seeed Studio XIAO Series Library:XIAO-nRF52840-DIP -> Module:MOUDLE14P-XIAO-DIP-SMD
Changed lines of the file:
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@@
 			)
 		)
-		(property "Footprint" "Seeed Studio XIAO Series Library:XIAO-nRF52840-DIP"
+		(property "Footprint" "Module:MOUDLE14P-XIAO-DIP-SMD"
 			(at 232.41 80.264 0)
 			(effects
