File: pcb_data/Assemble_L/Assemble_L.kicad_pcb (KiCad board)
At the start: 2 copper layers, 158.4 x 96.4 mm, 85 parts, among them J1 Conn_01x02, U1 XIAO-nRF52840

Commit message: tune hole positions
Parts:
- C1: value C -> GRM32EC81C476KE15L
- moved H2 0.60 mm to (128.6, 66.1)
- moved H3 0.60 mm to (185.7, 66.1)
- moved H5 0.60 mm to (128.6, 123.2)
- moved H6 0.60 mm to (185.7, 123.2)
- moved H8 0.60 mm to (142.9, 104.2)
Routing:
- net Net-(D0-2-K): track 162.2 -> 163.2 mm
Changed lines of the file:
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@@
 	(footprint "kbd_Hole:m2_Spacer_Hole"
 		(layer "F.Cu")
-		(at 185.737656 66.675056)
+		(at 185.737656 66.079743)
 		(descr "Mounting Hole 2.2mm, no annular, M2")
 		(tags "mounting hole 2.2mm no annular m2")
@@
 	(footprint "kbd_Hole:m2_Spacer_Hole"
 		(layer "F.Cu")
-		(at 185.737656 123.825104)
+		(at 185.737656 123.229791)
 		(descr "Mounting Hole 2.2mm, no annular, M2")
 		(tags "mounting hole 2.2mm no annular m2")
@@
 	(footprint "kbd_Hole:m2_Spacer_Hole"
 		(layer "F.Cu")
-		(at 128.587608 123.825104)
+		(at 128.587608 123.229791)
 		(descr "Mounting Hole 2.2mm, no annular, M2")
 		(tags "mounting hole 2.2mm no annular m2")
@@
 	(footprint "kbd_Hole:m2_Spacer_Hole"
 		(layer "F.Cu")
-		(at 142.87512 104.775088)
+		(at 142.87512 104.179775)
 		(descr "Mounting Hole 2.2mm, no annular, M2")
 		(tags "mounting hole 2.2mm no annular m2")
@@
 	(footprint "kbd_Hole:m2_Spacer_Hole"
 		(layer "F.Cu")
-		(at 128.587608 66.675056)
+		(at 128.587608 66.079743)
 		(descr "Mounting Hole 2.2mm, no annular, M2")
 		(tags "mounting hole 2.2mm no annular m2")
@@
 			)
 		)
-		(property "Value" "C"
+		(property "Value" "GRM32EC81C476KE15L"
 			(at 0 -2.3 0)
 			(layer "B.Fab")
@@
 	)
 	(segment
-		(start 137.160112 102.989149)
-		(end 135.969486 101.798523)
+		(start 141.684494 100.607897)
+		(end 139.303242 102.989149)
 		(width 0.5)
 		(layer "F.Cu")
@@
 	)
 	(segment
-		(start 127.15886 102.989149)
-		(end 134.77886 102.989149)
+		(start 137.160112 102.989149)
+		(end 135.969486 101.798523)
 		(width 0.5)
 		(layer "F.Cu")
@@
 	)
 	(segment
-		(start 144.661059 101.798523)
-		(end 141.089181 101.798523)
+		(start 127.15886 102.989149)
+		(end 134.77886 102.989149)
 		(width 0.5)
 		(layer "F.Cu")
@@
 	)
 	(segment
-		(start 139.898555 102.989149)
+		(start 139.303242 102.989149)
 		(end 137.160112 102.989149)
 		(width 0.5)
@@
 	)
 	(segment
-		(start 92.511637 103.584462)
-		(end 115.133531 103.584462)
+		(start 153.828876 102.989149)
+		(end 146.446998 102.989149)
 		(width 0.5)
 		(layer "F.Cu")
@@
 	)
 	(segment
-		(start 145.851685 102.989149)
-		(end 144.661059 101.798523)
+		(start 155.019502 101.798523)
+		(end 153.828876 102.989149)
 		(width 0.5)
 		(layer "F.Cu")
@@
 	)
 	(segment
-		(start 155.019502 101.798523)
-		(end 155.019502 102.036645)
+		(start 92.511637 103.584462)
+		(end 115.133531 103.584462)
 		(width 0.5)
 		(layer "F.Cu")
@@
 	)
 	(segment
-		(start 141.089181 101.798523)
-		(end 139.898555 102.989149)
+		(start 155.019502 101.798523)
+		(end 155.019502 102.036645)
 		(width 0.5)
 		(layer "F.Cu")
@@
 	)
 	(segment
-		(start 155.019502 101.798523)
-		(end 153.828876 102.989149)
+		(start 144.065746 100.607897)
+		(end 141.684494 100.607897)
+		(width 0.5)
+		(layer "F.Cu")
+		(net 3)
+	)
+	(segment
+		(start 146.446998 102.989149)
+		(end 144.065746 100.607897)
 		(width 0.5)
 		(layer "F.Cu")
@@
 	)
 	(segment
-		(start 153.828876 102.989149)
-		(end 145.851685 102.989149)
-		(width 0.5)
-		(layer "F.Cu")
-		(net 3)
-	)
-	(segment
 		(start 155.972006 102.989149)
 		(end 172.878892 102.989149)
@@
 	)
 	(segment
-		(start 102.631958 63.698491)
-		(end 103.822584 64.889117)
+		(start 125.01573 64.889117)
+		(end 127.396982 62.507865)
 		(width 0.5)
 		(layer "F.Cu")
@@
 	)
 	(segment
-		(start 127.396982 63.103178)
-		(end 130.373547 63.103178)
-		(width 0.5)
-		(layer "F.Cu")
-		(net 10)
-	)
-	(segment
-		(start 139.541364 64.889117)
-		(end 140.73199 63.698491)
+		(start 102.631958 63.698491)
+		(end 103.822584 64.889117)
 		(width 0.5)
 		(layer "F.Cu")
@@
 	(segment
 		(start 122.8726 64.889117)
-		(end 125.611043 64.889117)
+		(end 125.01573 64.889117)
 		(width 0.5)
 		(layer "F.Cu")
@@
 	)
 	(segment
-		(start 130.373547 63.103178)
-		(end 132.159486 64.889117)
+		(start 132.159486 64.889117)
+		(end 139.541364 64.889117)
 		(width 0.5)
 		(layer "F.Cu")
@@
 	)
 	(segment
-		(start 84.772568 64.889117)
-		(end 101.441332 64.889117)
+		(start 139.541364 64.889117)
+		(end 140.73199 63.698491)
 		(width 0.5)
 		(layer "F.Cu")
@@
 	)
 	(segment
-		(start 125.611043 64.889117)
-		(end 127.396982 63.103178)
+		(start 84.772568 64.889117)
+		(end 101.441332 64.889117)
 		(width 0.5)
 		(layer "F.Cu")
@@
 	)
 	(segment
-		(start 121.681974 63.698491)
-		(end 122.8726 64.889117)
+		(start 127.396982 62.507865)
+		(end 129.778234 62.507865)
 		(width 0.5)
 		(layer "F.Cu")
@@
 	)
 	(segment
-		(start 132.159486 64.889117)
-		(end 139.541364 64.889117)
+		(start 121.681974 63.698491)
+		(end 122.8726 64.889117)
 		(width 0.5)
 		(layer "F.Cu")
@@
 	)
 	(segment
+		(start 129.778234 62.507865)
+		(end 132.159486 64.889117)
+		(width 0.5)
+		(layer "F.Cu")
+		(net 10)
+	)
+	(segment
 		(start 83.581942 63.698491)
 		(end 84.772568 64.889117)
@@
 	)
 	(segment
-		(start 125.01573 64.293804)
-		(end 125.01573 67.57177)
-		(width 0.5)
-		(layer "B.Cu")
-		(net 42)
-	)
-	(segment
 		(start 149.423563 127.15886)
 		(end 149.423563 129.19386)
@@
 	(segment
 		(start 125.9635 59.451)
-		(end 125.9635 63.346034)
+		(end 125.9635 62.771735)
 		(width 0.5)
 		(layer "B.Cu")
@@
 	)
 	(segment
+		(start 125.01573 63.698491)
+		(end 125.01573 67.57177)
+		(width 0.5)
+		(layer "B.Cu")
+		(net 42)
+	)
+	(segment
 		(start 144.964911 124.95)
 		(end 139.075 124.95)
@@
 	)
 	(segment
+		(start 125.063221 63.651)
+		(end 125.01573 63.698491)
+		(width 0.5)
+		(layer "B.Cu")
+		(net 42)
+	)
+	(segment
+		(start 125.084235 63.651)
+		(end 125.063221 63.651)
+		(width 0.5)
+		(layer "B.Cu")
+		(net 42)
+	)
+	(segment
 		(start 146.00725 103.30725)
 		(end 146.00725 123.742547)
@@
 	)
 	(segment
-		(start 146.00725 123.742547)
-		(end 146.089807 123.825104)
+		(start 125.9635 62.771735)
+		(end 125.084235 63.651)
 		(width 0.5)
 		(layer "B.Cu")
@@
 	)
 	(segment
-		(start 125.9635 63.346034)
-		(end 125.01573 64.293804)
+		(start 125.01573 67.57177)
+		(end 124.7875 67.8)
 		(width 0.5)
 		(layer "B.Cu")
@@
 	)
 	(segment
-		(start 125.01573 67.57177)
-		(end 124.7875 67.8)
+		(start 146.00725 123.742547)
+		(end 146.089807 123.825104)
 		(width 0.5)
 		(layer "B.Cu")
@@
 	)
 	(via
-		(at 128.5875 61.9125)
+		(at 128.587608 61.317239)
 		(size 0.6)
 		(drill 0.3)

Commit message: fix power line pattern width
Changed lines of the file:
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@@
 		(start 52.601605 79.771942)
 		(end 52.601605 71.43756)
-		(width 1)
+		(width 0.75)
 		(layer "B.Cu")
 		(net 46)
@@
 		(start 52.601605 71.43756)
 		(end 56.107857 67.931308)
-		(width 1)
+		(width 0.75)
 		(layer "B.Cu")
 		(net 46)
@@
 		(start 56.107857 56.70317)
 		(end 56.107857 63.103178)
-		(width 1)
+		(width 0.75)
 		(layer "B.Cu")
 		(net 46)
@@
 		(start 52.705 57.30925)
 		(end 52.705 56.321422)
-		(width 1)
+		(width 0.75)
 		(layer "B.Cu")
 		(net 46)
@@
 		(start 55.364109 55.959422)
 		(end 56.107857 56.70317)
-		(width 1)
+		(width 0.75)
 		(layer "B.Cu")
 		(net 46)
@@
 		(start 52.705 56.321422)
 		(end 53.067 55.959422)
-		(width 1)
+		(width 0.75)
 		(layer "B.Cu")
 		(net 46)
@@
 		(start 56.107857 67.931308)
 		(end 56.107857 63.103178)
-		(width 1)
+		(width 0.75)
 		(layer "B.Cu")
 		(net 46)
@@
 		(start 53.067 55.959422)
 		(end 55.364109 55.959422)
-		(width 1)
+		(width 0.75)
 		(layer "B.Cu")
 		(net 46)
@@
 		(start 50.601605 79.771942)
 		(end 50.601605 69.651621)
-		(width 1)
+		(width 0.75)
 		(layer "B.Cu")
 		(net 48)
@@
 		(start 52.692986 62.813307)
 		(end 52.692986 59.732957)
-		(width 1)
+		(width 0.75)
 		(layer "B.Cu")
 		(net 48)
@@
 		(start 52.982857 67.270369)
 		(end 52.982857 63.103178)
-		(width 1)
+		(width 0.75)
 		(layer "B.Cu")
 		(net 48)
@@
 		(start 52.982857 63.103178)
 		(end 52.692986 62.813307)
-		(width 1)
+		(width 0.75)
 		(layer "B.Cu")
 		(net 48)
@@
 		(start 50.601605 69.651621)
 		(end 52.982857 67.270369)
-		(width 1)
+		(width 0.75)
 		(layer "B.Cu")
 		(net 48)

Commit message: tune hole position near by xiao
Parts:
- moved H7 12.7 mm to (60.7, 80.4)
Routing:
- net IO 2: track 158.2 -> 159.4 mm
Changed lines of the file:
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@@
 	(footprint "kbd_Hole:m2_Spacer_Hole"
 		(layer "F.Cu")
-		(at 51.196918 88.701637)
+		(at 60.721926 80.367255)
 		(descr "Mounting Hole 2.2mm, no annular, M2")
 		(tags "mounting hole 2.2mm no annular m2")
@@
 	)
 	(segment
-		(start 57.745361 98.821958)
-		(end 58.935987 100.012584)
+		(start 46.327 70.13952)
+		(end 46.327 54.03662)
 		(width 0.5)
 		(layer "F.Cu")
@@
 	)
 	(segment
-		(start 58.935987 100.012584)
-		(end 62.507865 100.012584)
+		(start 65.48443 83.105698)
+		(end 65.48443 80.367255)
 		(width 0.5)
 		(layer "F.Cu")
@@
 	)
 	(segment
-		(start 63.936613 83.105698)
-		(end 59.5313 87.511011)
+		(start 65.48443 80.367255)
+		(end 61.912552 76.795377)
 		(width 0.5)
 		(layer "F.Cu")
@@
 	)
 	(segment
-		(start 65.48443 83.105698)
-		(end 65.48443 80.962568)
+		(start 57.745361 98.821958)
+		(end 58.935987 100.012584)
 		(width 0.5)
 		(layer "F.Cu")
@@
 	)
 	(segment
-		(start 60.483804 106.322905)
-		(end 65.48443 111.323531)
+		(start 52.982857 76.795377)
+		(end 46.327 70.13952)
 		(width 0.5)
 		(layer "F.Cu")
@@
 	)
 	(segment
-		(start 48.45237 51.91125)
-		(end 49.53 51.91125)
+		(start 46.327 54.03662)
+		(end 48.45237 51.91125)
 		(width 0.5)
 		(layer "F.Cu")
@@
 	)
 	(segment
-		(start 62.507865 100.012584)
-		(end 63.936613 98.583836)
+		(start 61.912552 76.795377)
+		(end 52.982857 76.795377)
 		(width 0.5)
 		(layer "F.Cu")
@@
 	)
 	(segment
-		(start 59.5313 106.322905)
-		(end 60.483804 106.322905)
+		(start 58.935987 100.012584)
+		(end 62.507865 100.012584)
 		(width 0.5)
 		(layer "F.Cu")
@@
 	)
 	(segment
-		(start 59.5313 121.801043)
-		(end 59.5313 120.015104)
+		(start 63.936613 83.105698)
+		(end 59.5313 87.511011)
 		(width 0.5)
 		(layer "F.Cu")
@@
 	)
 	(segment
-		(start 63.936613 98.583836)
-		(end 65.48443 98.583836)
+		(start 60.483804 106.322905)
+		(end 65.48443 111.323531)
 		(width 0.5)
 		(layer "F.Cu")
@@
 	)
 	(segment
-		(start 59.5313 90.844767)
-		(end 57.745361 92.630706)
+		(start 62.507865 100.012584)
+		(end 63.936613 98.583836)
 		(width 0.5)
 		(layer "F.Cu")
@@
 	)
 	(segment
-		(start 65.48443 83.105698)
-		(end 63.936613 83.105698)
+		(start 59.5313 106.322905)
+		(end 60.483804 106.322905)
 		(width 0.5)
 		(layer "F.Cu")
@@
 	)
 	(segment
-		(start 63.103178 78.581316)
-		(end 54.768796 78.581316)
+		(start 59.5313 121.801043)
+		(end 59.5313 120.015104)
 		(width 0.5)
 		(layer "F.Cu")
@@
 	)
 	(segment
-		(start 54.768796 78.581316)
-		(end 46.327 70.13952)
+		(start 63.936613 98.583836)
+		(end 65.48443 98.583836)
 		(width 0.5)
 		(layer "F.Cu")
@@
 	)
 	(segment
-		(start 59.5313 106.322905)
-		(end 59.5313 104.536966)
+		(start 59.5313 90.844767)
+		(end 57.745361 92.630706)
 		(width 0.5)
 		(layer "F.Cu")
@@
 	)
 	(segment
-		(start 59.5313 120.015104)
-		(end 65.48443 114.061974)
+		(start 65.48443 83.105698)
+		(end 63.936613 83.105698)
 		(width 0.5)
 		(layer "F.Cu")
@@
 	)
 	(segment
-		(start 46.327 70.13952)
-		(end 46.327 54.03662)
+		(start 59.5313 106.322905)
+		(end 59.5313 104.536966)
 		(width 0.5)
 		(layer "F.Cu")
@@
 	)
 	(segment
-		(start 46.327 54.03662)
-		(end 48.45237 51.91125)
+		(start 59.5313 120.015104)
+		(end 65.48443 114.061974)
 		(width 0.5)
 		(layer "F.Cu")
@@
 	)
 	(segment
-		(start 65.48443 80.962568)
-		(end 63.103178 78.581316)
+		(start 48.45237 51.91125)
+		(end 49.53 51.91125)
 		(width 0.5)
 		(layer "F.Cu")
@@
 	)
 	(segment
-		(start 72.032873 76.200064)
-		(end 82.682809 86.85)
+		(start 54.617743 75.604751)
+		(end 71.43756 75.604751)
 		(width 0.5)
 		(layer "F.Cu")
@@
 	)
 	(segment
-		(start 47.028 68.015008)
-		(end 55.213056 76.200064)
+		(start 82.682809 86.85)
+		(end 84.30625 86.85)
 		(width 0.5)
 		(layer "F.Cu")
@@
 	)
 	(segment
-		(start 47.028 56.11825)
-		(end 47.028 68.015008)
+		(start 71.43756 75.604751)
+		(end 82.682809 86.85)
 		(width 0.5)
 		(layer "F.Cu")
@@
 	)
 	(segment
-		(start 55.213056 76.200064)
-		(end 72.032873 76.200064)
+		(start 47.028 56.11825)
+		(end 47.028 68.015008)
 		(width 0.5)
 		(layer "F.Cu")
@@
 	)
 	(segment
-		(start 82.682809 86.85)
-		(end 84.30625 86.85)
+		(start 47.028 68.015008)
+		(end 54.617743 75.604751)
 		(width 0.5)
 		(layer "F.Cu")
@@
 	)
 	(segment
+		(start 118.467287 86.677576)
+		(end 118.467287 79.771942)
+		(width 0.5)
+		(layer "B.Cu")
+		(net 41)
+	)
+	(segment
 		(start 106.9135 59.451)
 		(end 106.9135 66.624)
@@
 	)
 	(segment
+		(start 118.467287 79.771942)
+		(end 106.495345 67.8)
+		(width 0.5)
+		(layer "B.Cu")
+		(net 41)
+	)
+	(segment
 		(start 120.848539 89.058828)
-		(end 120.848539 82.911039)
+		(end 118.467287 86.677576)
 		(width 0.5)
 		(layer "B.Cu")
@@
 	)
 	(segment
+		(start 105.7375 68.611703)
+		(end 105.7375 67.8)
+		(width 0.5)
+		(layer "B.Cu")
+		(net 41)
+	)
+	(segment
 		(start 132.833486 104.420986)
 		(end 134.3125 105.9)
@@
 	)
 	(segment
-		(start 106.9135 66.624)
+		(start 106.495345 67.8)
 		(end 105.7375 67.8)
 		(width 0.5)
@@
 	)
 	(segment
-		(start 130.299 95.369159)
-		(end 130.299 99.686037)
+		(start 106.9135 66.624)
+		(end 105.7375 67.8)
 		(width 0.5)
 		(layer "B.Cu")
@@
 	)
 	(segment
-		(start 120.848539 82.911039)
-		(end 105.7375 67.8)
+		(start 130.299 95.369159)
+		(end 130.299 99.686037)
 		(width 0.5)
 		(layer "B.Cu")
@@
 	)
 	(via
-		(at 117.871974 82.153194)
+		(at 116.681348 85.129759)
 		(size 0.6)
 		(drill 0.3)
@@
 	)
 	(via
-		(at 64.29375 78.58125)
+		(at 66.675056 78.58125)
 		(size 0.6)
 		(drill 0.3)

Commit message: fix position of mounting hole
Parts:
- moved H4 4.29 mm to (73.8, 121.4)
- moved H1 3.37 mm to (73.8, 69.1)
Routing:
- net Net-(D1-0-K): track 157.4 -> 159.2 mm
Changed lines of the file:
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@@
 	(footprint "kbd_Hole:m2_Spacer_Hole"
 		(layer "F.Cu")
-		(at 71.43756 66.675056)
+		(at 73.818812 69.056308)
 		(descr "Mounting Hole 2.2mm, no annular, M2")
 		(tags "mounting hole 2.2mm no annular m2")
@@
 	(footprint "kbd_Hole:m2_Spacer_Hole"
 		(layer "F.Cu")
-		(at 70.246934 123.825104)
+		(at 73.818812 121.443852)
 		(descr "Mounting Hole 2.2mm, no annular, M2")
 		(tags "mounting hole 2.2mm no annular m2")
@@
 	)
 	(segment
-		(start 65.48443 88.106324)
-		(end 67.865682 85.725072)
+		(start 72.628186 72.628186)
+		(end 75.604751 72.628186)
 		(width 0.5)
 		(layer "B.Cu")
@@
 	)
 	(segment
-		(start 67.865682 77.379751)
-		(end 81.546942 63.698491)
+		(start 77.39069 67.865682)
+		(end 81.546942 63.70943)
 		(width 0.5)
 		(layer "B.Cu")
@@
 	)
 	(segment
+		(start 67.865682 77.379751)
+		(end 67.876621 77.379751)
+		(width 0.5)
+		(layer "B.Cu")
+		(net 10)
+	)
+	(segment
 		(start 87.511011 58.578796)
 		(end 87.511011 56.543796)
@@
 	)
 	(segment
+		(start 67.876621 77.379751)
+		(end 72.628186 72.628186)
+		(width 0.5)
+		(layer "B.Cu")
+		(net 10)
+	)
+	(segment
 		(start 81.546942 63.698491)
 		(end 83.581942 63.698491)
@@
 	)
 	(segment
+		(start 77.39069 70.842247)
+		(end 77.39069 67.865682)
+		(width 0.5)
+		(layer "B.Cu")
+		(net 10)
+	)
+	(segment
+		(start 75.604751 72.628186)
+		(end 77.39069 70.842247)
+		(width 0.5)
+		(layer "B.Cu")
+		(net 10)
+	)
+	(segment
+		(start 81.546942 63.70943)
+		(end 81.546942 63.698491)
+		(width 0.5)
+		(layer "B.Cu")
+		(net 10)
+	)
+	(segment
+		(start 65.48443 88.106324)
+		(end 67.865682 85.725072)
+		(width 0.5)
+		(layer "B.Cu")
+		(net 10)
+	)
+	(segment
 		(start 87.511011 58.578796)
 		(end 86.523183 58.578796)
@@
 	)
 	(segment
-		(start 143.176505 68.460995)
-		(end 143.8375 67.8)
+		(start 50.919051 64.61125)
+		(end 58.340674 72.032873)
 		(width 0.5)
 		(layer "F.Cu")
@@
 	)
 	(segment
-		(start 79.242311 67.8)
-		(end 123.164109 67.8)
+		(start 125.611043 68.460995)
+		(end 127.396982 70.246934)
 		(width 0.5)
 		(layer "F.Cu")
@@
 	)
 	(segment
-		(start 127.396982 70.246934)
-		(end 130.373547 70.246934)
+		(start 123.164109 67.8)
+		(end 123.825104 68.460995)
 		(width 0.5)
 		(layer "F.Cu")
@@
 	)
 	(segment
-		(start 125.611043 68.460995)
-		(end 127.396982 70.246934)
+		(start 143.176505 68.460995)
+		(end 143.8375 67.8)
 		(width 0.5)
 		(layer "F.Cu")
@@
 	)
 	(segment
-		(start 49.53 64.61125)
-		(end 50.919051 64.61125)
+		(start 58.340674 72.032873)
+		(end 75.604751 72.032873)
 		(width 0.5)
 		(layer "F.Cu")
@@
 	)
 	(segment
-		(start 132.159486 68.460995)
-		(end 143.176505 68.460995)
+		(start 123.825104 68.460995)
+		(end 125.611043 68.460995)
 		(width 0.5)
 		(layer "F.Cu")
@@
 	)
 	(segment
-		(start 123.164109 67.8)
-		(end 123.825104 68.460995)
+		(start 49.53 64.61125)
+		(end 50.919051 64.61125)
 		(width 0.5)
 		(layer "F.Cu")
@@
 	)
 	(segment
-		(start 123.825104 68.460995)
-		(end 125.611043 68.460995)
+		(start 127.396982 70.246934)
+		(end 130.373547 70.246934)
 		(width 0.5)
 		(layer "F.Cu")
@@
 	)
 	(segment
-		(start 75.604751 71.43756)
-		(end 79.242311 67.8)
+		(start 75.604751 72.032873)
+		(end 79.837624 67.8)
 		(width 0.5)
 		(layer "F.Cu")
@@
 	)
 	(segment
-		(start 57.745361 71.43756)
-		(end 75.604751 71.43756)
+		(start 132.159486 68.460995)
+		(end 143.176505 68.460995)
 		(width 0.5)
 		(layer "F.Cu")
@@
 	)
 	(segment
-		(start 50.919051 64.61125)
-		(end 57.745361 71.43756)
+		(start 79.837624 67.8)
+		(end 123.164109 67.8)
 		(width 0.5)
 		(layer "F.Cu")
@@
 	)
 	(via
-		(at 73.81875 119.0625)
+		(at 74.414125 117.276661)
 		(size 0.6)
 		(drill 0.3)

Commit message: fix hole footprint and number
Parts:
- renumbered H8 to H7, H7 to H8
Changed lines of the file:
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@@
 		(descr "Mounting Hole 2.2mm, no annular, M2")
 		(tags "mounting hole 2.2mm no annular m2")
-		(property "Reference" "H7"
+		(property "Reference" "H8"
 			(at 0 -3.2 0)
 			(layer "F.Fab")
@@
 		(descr "Mounting Hole 2.2mm, no annular, M2")
 		(tags "mounting hole 2.2mm no annular m2")
-		(property "Reference" "H8"
+		(property "Reference" "H7"
 			(at 0 -3.2 0)
 			(layer "F.Fab")
